File: keeb.kicad_pcb (KiCad board)
At the start: 2 copper layers, 345 x 120 mm, 204 parts, among them SW1 Push, SW10 Push, SW11 Push, SW12 Push, SW13 Push, SW14 Push, SW15 Push, SW16 Push, SW17 Push, SW18 Push, SW19 Push, SW2 Push, SW20 Push, SW21 Push, SW22 Push, SW23 Push, SW24 Push, SW25 Push, SW26 Push, SW27 Push, SW28 Push, SW29 Push, SW3 Push, SW30 Push, SW31 Push, SW32 Push, SW33 Push, SW34 Push, SW35 Push, SW36 Push, SW37 Push, SW38 Push, SW39 Push, SW4 Push, SW40 Push, SW41 Push, SW42 Push, SW43 Push, SW44 Push, SW45 Push, SW46 Push, SW47 Push, SW48 Push, SW49 Push, SW5 Push, SW50 Push, SW51 Push, SW52 Push, SW53 Push, SW54 Push, SW55 Push, SW56 Push, SW57 Push, SW58 Push, SW59 Push, SW6 Push, SW60 Push, SW61 Push, SW62 Push, SW63 Push, SW64 Push, SW65 Push, SW66 Push, SW67 Push, SW68 Push, SW69 Push, SW7 Push, SW70 Push, SW71 Push, SW72 Push, SW73 Push, SW74 Push, SW75 Push, SW76 Push, SW77 Push, SW78 Push, SW79 Push, SW8 Push, SW80 Push, SW81 Push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

Commit message: a
Parts:
- SW1, SW28, SW30, SW45, SW57, SW59, SW70, SW76, SW77: footprint keys:SW_MX_LowProfile_THT -> keys:SW_MX_LowProfile_THT_NoKey
