File: keeb.kicad_sch (KiCad schematic)
At the start: 207 parts, among them SW1 Push, SW10 Push, SW11 Push, SW12 Push, SW13 Push, SW14 Push, SW15 Push, SW16 Push, SW17 Push, SW18 Push, SW19 Push, SW2 Push, SW20 Push, SW21 Push, SW22 Push, SW23 Push, SW24 Push, SW25 Push, SW26 Push, SW27 Push, SW28 Push, SW29 Push, SW3 Push, SW30 Push, SW31 Push, SW32 Push, SW33 Push, SW34 Push, SW35 Push, SW36 Push, SW37 Push, SW38 Push, SW39 Push, SW4 Push, SW40 Push, SW41 Push, SW42 Push, SW43 Push, SW44 Push, SW45 Push, SW46 Push, SW47 Push, SW48 Push, SW49 Push, SW5 Push, SW50 Push, SW51 Push, SW52 Push, SW53 Push, SW54 Push, SW55 Push, SW56 Push, SW57 Push, SW58 Push, SW59 Push, SW6 Push, SW60 Push, SW61 Push, SW62 Push, SW63 Push, SW64 Push, SW65 Push, SW66 Push, SW67 Push, SW68 Push, SW69 Push, SW7 Push, SW70 Push, SW71 Push, SW72 Push, SW73 Push, SW74 Push, SW75 Push, SW76 Push, SW77 Push, SW78 Push, SW79 Push, SW8 Push, SW80 Push, SW81 Push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

Commit message: a
Other:
- note added: "Esc 1.5U"
- note removed: "Esc 1U"
Changed lines of the file:
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@@
 		)
 	)
-	(text "Esc 1U"
+	(text "Esc 1.5U"
 		(exclude_from_sim no)
 		(at 30.48 62.738 0)

Commit message: csv init
Other:
- note added: "to-do: pbt keycaps MX LP Red - 100 ($44 Taobao)"
- note removed: "to-do: update the entire pcb pbt keycaps MX LP Red - 100 ($44 Taobao)"
Changed lines of the file:
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@@
 		)
 	)
-	(text "to-do:\nupdate the entire pcb\npbt keycaps\nMX LP Red - 100 ($44 Taobao)\n"
+	(text "to-do:\npbt keycaps\nMX LP Red - 100 ($44 Taobao)\n"
 		(exclude_from_sim no)
 		(at 131.318 170.942 0)

Commit message: finalised production render and casing
Other:
- added sheet Plate (plate.kicad_sch)
- added sheet main_pcb (main_pcb.kicad_sch)
Changed lines of the file:
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@@
+		)
+	)
+	(sheet
+		(at 398.78 3.81)
+		(size 12.7 3.81)
+		(exclude_from_sim no)
+		(in_bom yes)
+		(on_board yes)
+		(dnp no)
+		(fields_autoplaced yes)
+		(stroke
+			(width 0.1524)
+			(type solid)
+		)
+		(fill
+			(color 0 0 0 0)
+		)
+		(property "Sheetname" "main_pcb"
+			(at 398.78 3.0984 0)
+			(show_name no)
+			(do_not_autoplace no)
+			(effects
+				(font
+					(size 1.27 1.27)
+				)
+				(justify left bottom)
+			)
+		)
+		(property "Sheetfile" "main_pcb.kicad_sch"
+			(at 398.78 8.2046 0)
+			(show_name no)
+			(do_not_autoplace no)
+			(effects
+				(font
+					(size 1.27 1.27)
+				)
+				(justify left top)
+			)
+		)
+		(instances
+			(project "keeb"
+				(path "/98fcfa59-6c4c-4e6f-8937-468a9e43a4b3"
+					(page "2")
+				)
+			)
+		)
+	)
+	(sheet
+		(at 160.02 -147.32)
+		(size 12.7 3.81)
+		(exclude_from_sim no)
+		(in_bom yes)
+		(on_board yes)
+		(dnp no)
+		(fields_autoplaced yes)
+		(stroke
+			(width 0.1524)
+			(type solid)
+		)
+		(fill
+			(color 0 0 0 0)
+		)
+		(property "Sheetname" "Plate"
+			(at 160.02 -148.0316 0)
+			(show_name no)
+			(do_not_autoplace no)
+			(effects
+				(font
+					(size 1.27 1.27)
+				)
+				(justify left bottom)
+			)
+		)
+		(property "Sheetfile" "plate.kicad_sch"
+			(at 160.02 -142.9254 0)
+			(show_name no)
+			(do_not_autoplace no)
+			(effects
+				(font
+					(size 1.27 1.27)
+				)
+				(justify left top)
+			)
+		)
+		(instances
+			(project "keeb"
+				(path "/98fcfa59-6c4c-4e6f-8937-468a9e43a4b3"
+					(page "3")
+				)
+			)
 		)
 	)
